File: Example-Palette/NYCpalette.kicad_pcb (KiCad board)
At the start: 2 copper layers, 85.7 x 54 mm, 1 part

Commit message: Completed the Palette tapeout
Parts:
- added REF**: MountingHole_2.2mm_M2_Pad_Via, MountingHole:MountingHole_2.2mm_M2_Pad_Via, F.Cu at (77.7, 99.6)
- added REF**: MountingHole_2.2mm_M2_Pad_Via, MountingHole:MountingHole_2.2mm_M2_Pad_Via, F.Cu at (156.0, 52.8)
- added REF**: MountingHole_2.2mm_M2_Pad_Via, MountingHole:MountingHole_2.2mm_M2_Pad_Via, F.Cu at (77.7, 52.8)
- added REF**: MountingHole_2.2mm_M2_Pad_Via, MountingHole:MountingHole_2.2mm_M2_Pad_Via, F.Cu at (156.0, 99.6)
- moved svg2mod 0.51 mm to (94.5, 53.3)
Other:
- board text added: "B.Cu"
- board text added: "B.Cu + B.Mask"
- board text added: "B.Mask"
- board text added: "B.SilkS"
- board text added: "F.Cu"
- board text added: "F.Cu + F.Mask"
- board text added: "F.Mask"
- board text added: "F.SilkS"
- board text added: "Palette-v1 A. Tait 5/26"
