File: Example-Zoo/pcb-artwork-zoo.kicad_pcb (KiCad board)
At the start: 2 copper layers, 5 parts

Commit message: Zoo tapeout
Parts:
- removed the svg2mod at (275.6, 12.7)
- svg2mod: moved to B.Cu
- moved svg2mod 104.1 mm to (127.1, 74.7), turned to 180 degrees
- moved svg2mod 69.0 mm to (169.0, 127.1)
- moved svg2mod 2.10 mm to (164.4, 50.3)
Other:
- board outline added: 104.1 x 106.7 mm
- board text added: "artwork-zoo-v1 A. Tait 5/26"
